Commit message: Fixed Multple Joint Publishers

File: src/arm_pkg/description/robot.urdf.xacro (robot description, xacro)
@@ -27,5 +27,5 @@
     <parent link="base_link"/>
     <child link="link1"/>
-    <origin rpy="0 0 0" xyz="0 0 0.15"/>
+    <origin rpy="0 0 0" xyz="0 0 0.1519"/>
   </joint>
   <!-- Joint 2 -->
@@ -34,5 +34,5 @@
     <parent link="link1"/>
     <child link="link2"/>
-    <origin rpy="1.57075 0 0" xyz="0 0 0.3"/>
+    <origin rpy="1.57075 0 0" xyz="0 0 0.24365"/>
   </joint>
   <!-- Joint 3 -->
@@ -41,5 +41,5 @@
     <parent link="link2"/>
     <child link="link3"/>
-    <origin rpy="0 0 1.57075" xyz="0 1 0"/>
+    <origin rpy="0 0 1.57075" xyz="0 0.21325 0"/>
   </joint>
   <!-- Joint 4 -->
@@ -48,5 +48,5 @@
     <parent link="link3"/>
     <child link="link4"/>
-    <origin rpy="0 0 0" xyz="0.5 0 0"/>
+    <origin rpy="0 0 0" xyz="0.11235 0 0"/>
   </joint>
   <!-- Joint 5 -->
@@ -55,5 +55,5 @@
     <parent link="link4"/>
     <child link="link5"/>
-    <origin rpy="1.57075 0 1.57075" xyz="0 0 -0.4"/>
+    <origin rpy="1.57075 0 1.57075" xyz="0 0 -0.08535"/>
   </joint>
   <!-- Joint 6 -->
@@ -62,5 +62,5 @@
     <parent link="link5"/>
     <child link="link6"/>
-    <origin rpy="1.57075 0 0" xyz="0 0 0.4"/>
+    <origin rpy="1.57075 0 0" xyz="0 0 0.0819"/>
   </joint>
   <!-- Link 1 -->
@@ -68,5 +68,5 @@
     <visual>
       <geometry>
-        <cylinder length="0.2" radius="0.2"/>
+        <cylinder length="0.05" radius="0.05"/>
       </geometry>
       <material name="black"/>
@@ -78,5 +78,5 @@
       <origin rpy="0 0 1.57075" xyz="0 0 0"/>
       <geometry>
-        <cylinder length="0.2" radius="0.2"/>
+        <cylinder length="0.05" radius="0.05"/>
       </geometry>
       <material name="black"/>
@@ -88,5 +88,5 @@
       <origin rpy="0 0 1.57075" xyz="0 0 0"/>
       <geometry>
-        <cylinder length="0.2" radius="0.2"/>
+        <cylinder length="0.05" radius="0.05"/>
       </geometry>
       <material name="black"/>
@@ -98,5 +98,5 @@
       <origin rpy="0 0 1.57075" xyz="0 0 0"/>
       <geometry>
-        <cylinder length="0.2" radius="0.2"/>
+        <cylinder length="0.05" radius="0.05"/>
       </geometry>
       <material name="black"/>
@@ -108,5 +108,5 @@
       <origin rpy="0 0 1.57075" xyz="0 0 0"/>
       <geometry>
-        <cylinder length="0.2" radius="0.2"/>
+        <cylinder length="0.05" radius="0.05"/>
       </geometry>
       <material name="black"/>
@@ -118,5 +118,5 @@
       <origin rpy="0 0 1.57075" xyz="0 0 0"/>
       <geometry>
-        <cylinder length="0.2" radius="0.2"/>
+        <cylinder length="0.05" radius="0.05"/>
       </geometry>
       <material name="black"/>

Commit message: Added Joint Subscriber

File: src/arm_pkg/description/robot.urdf.xacro (robot description, xacro)
@@ -27,5 +27,5 @@
     <parent link="base_link"/>
     <child link="link1"/>
-    <origin rpy="0 0 0" xyz="0 0 0.1519"/>
+    <origin rpy="0 0 0" xyz="0 0 0"/>
   </joint>
   <!-- Joint 2 -->
@@ -34,5 +34,5 @@
     <parent link="link1"/>
     <child link="link2"/>
-    <origin rpy="1.57075 0 0" xyz="0 0 0.24365"/>
+    <origin rpy="1.57075 0 0" xyz="0 0 0.1519"/>
   </joint>
   <!-- Joint 3 -->
@@ -41,5 +41,5 @@
     <parent link="link2"/>
     <child link="link3"/>
-    <origin rpy="0 0 1.57075" xyz="0 0.21325 0"/>
+    <origin rpy="0 0 1.57075" xyz="0 -0.24365 0"/>
   </joint>
   <!-- Joint 4 -->
@@ -48,5 +48,5 @@
     <parent link="link3"/>
     <child link="link4"/>
-    <origin rpy="0 0 0" xyz="0.11235 0 0"/>
+    <origin rpy="0 0 0" xyz="-0.21325 0 0"/>
   </joint>
   <!-- Joint 5 -->
@@ -55,5 +55,5 @@
     <parent link="link4"/>
     <child link="link5"/>
-    <origin rpy="1.57075 0 1.57075" xyz="0 0 -0.08535"/>
+    <origin rpy="1.57075 0 1.57075" xyz="0 0 0.11235"/>
   </joint>
   <!-- Joint 6 -->
@@ -62,5 +62,12 @@
     <parent link="link5"/>
     <child link="link6"/>
-    <origin rpy="1.57075 0 0" xyz="0 0 0.0819"/>
+    <origin rpy="1.57075 0 0" xyz="0 0 0.08535"/>
+  </joint>
+  <!-- Joint 7 -->
+  <joint name="joint7" type="fixed">
+    <axis rpy="0 0 0" xyz="0 0 1"/>
+    <parent link="link6"/>
+    <child link="end"/>
+    <origin rpy="0 0 0" xyz="0 0 0.0819"/>
   </joint>
   <!-- Link 1 -->
@@ -123,3 +130,13 @@
     </visual>
   </link>
+  <!-- End Effector -->
+  <link name="end">
+    <visual>
+      <origin rpy="0 0 1.57075" xyz="0 0 0"/>
+      <geometry>
+        <cylinder length="0.01" radius="0.05"/>
+      </geometry>
+      <material name="black"/>
+    </visual>
+  </link>
 </robot>
